File: hardware/pidp8i/PDP8.sch (KiCad schematic (older format))
At the start: 174 parts, among them M1 M, M2 M, M3 M, M4 M, M5 M, M6 M, M7 M, P1 RASPI_MODEL_B_PLUS_GPIO, P2 UDN2981A, P3 EXPANSION_20X2, P5 SERIAL 5V TTL, SW1 DF1, SW10 SR4, SW11 SR5, SW12 SR6, SW13 SR7, SW14 SR8, SW15 SR9, SW16 SR10, SW17 SR11, SW18 SR12, SW19 START, SW2 DF2, SW20 LOAD_ADD, SW21 DEP, SW22 EXAM, SW23 CONT, SW24 STOP, SW25 SING_STEP, SW26 SING_INST, SW3 DF3, SW4 IF1, SW5 IF2, SW6 IF3, SW7 SR1, SW8 SR2, SW9 SR3

Commit message: Updated the PiDP-8/I KiCad hardware files to the 2019 kit version.
FossilOrigin-Name: 4be67ee54444fb936511be7e97eda3a59b6e85471df8ba7478f6c0bcefba58b8
Parts:
- removed J_COL1, J_COL2: CONN_3, symbol CONN_3
- removed P3: EXPANSION_20X2, symbol CONN_20X2
- removed P5: SERIAL 5V TTL, symbol CONN_4
- removed R_S1: 300, ~, symbol R
- removed R_S2: 620, ~, symbol R
- added P3: CONN_4, symbol CONN_4
Connections:
- net labels added: i2cgnd, scl, sda
- net labels removed: RX, SPARE_IO, TX, col1a, col2a
- wire segments 319 -> 281
- no-connect marks 41 -> 42
Other:
- note removed: "2 Expansion ports"
- note removed: "5V TTL compatible serial port (option). \nWarning: requires mod on RPi (remove R23/24)\n & trace cut/jumper on PiDP\nWarning: do not install resistors R_S1/R_S2 until \n this mod has been done\n"
- note removed: "Serial Port Option jumper.\nWarning: enabling Serial Port requires modification on Raspberry Pi.\nWarning2: circuit board traces 1-2 are added\non the PiDP circuit board to enable default option \n(no serial port, unmodified RPI). Cut traces and \njumper 2-3 to enable serial port after \nmodifying the RPi."
- moved on the sheet: R1, R2
